File: 0011_Distance_Module_TMF8828.kicad_sch (KiCad schematic)
At the start: 10 parts, among them IC1 TMF8820-1AM

Commit message: Add files via upload
Parts:
- added D1: LED, LED_SMD:LED_0603_1608Metric, symbol Device:LED
- added R7: 470r, Resistor_SMD:R_0603_1608Metric, symbol Device:R
- added U1: ~, Moduler_:pin_header, symbol moduler_pin:air
- C1, C2, C3: footprint (none) -> Capacitor_SMD:C_0603_1608Metric
- IC1: footprint TMF88201AM -> TMF8820:TMF88201AM
- R1, R2, R3, R4, R5, R6: footprint (none) -> Resistor_SMD:R_0603_1608Metric
Connections:
- net EN: now also U1.12
- net GND: now also D1.1 (K), U1.9
- net GPIO0: now also U1.14
- net GPIO1: now also U1.15
- net INT: now also U1.13
- net SCL: now also U1.5
- net SDA: now also U1.6
- net VCC renamed +3V3
- net +3V3: now also R7.1, U1.8
- new net: D1.2 (A), R7.2
- no-connect marks 0 -> 10
Other:
- note added: "AIR PIN"
- note added: "SENSOR"
- moved on the sheet: C1, C2, C3, IC1, R1, R2, R3, R4, R5, R6
